Commit message: added arms and changed colors

File: my_robot_urdf/urdf/robo.xacro (robot description, xacro)
@@ -1,4 +1,152 @@
 <?xml version='1.0'?>
 <robot name="robo" xmlns:xacro="http://www.ros.org/wiki/xacro">
+  <xacro:include filename="$(find my_robot_urdf)/urdf/robo.gazebo" />
+  <gazebo reference="left_wheel">
+    <material>Gazebo/Black</material>
+  </gazebo>
+  <gazebo reference="right_wheel">
+    <material>Gazebo/Black</material>
+  </gazebo>
+  <gazebo reference="camera">
+    <material>Gazebo/Black</material>
+  </gazebo>
+  <gazebo reference="hokuyo">
+    <material>Gazebo/Red</material>
+  </gazebo>
+  <gazebo reference="leftarm">
+    <material>Gazebo/Grey</material>
+  </gazebo>
+  <gazebo reference="rightarm">
+    <material>Gazebo/Grey</material>
+  </gazebo>
+  <gazebo reference="chassis">
+    <material>Gazebo/Yellow</material>
+  </gazebo>
+  <link name="robot_footprint"></link>
+  <joint name="robot_footprint_joint" type="fixed">
+    <origin xyz="0 0 0" rpy="0 0 0" />
+    <parent link="robot_footprint"/>
+    <child link="chassis" />
+  </joint>
+  <joint name="camera_joint" type="fixed">
+    <origin xyz="0.26 0 0.1" rpy="0 0 0" />
+    <parent link="chassis"/>
+    <child link="camera" />
+    <axis xyz="0 1 0"/>
+  </joint>
+  <joint name="hokuyo_joint" type="fixed">
+    <origin xyz="0.2 0 0.2" rpy="0 0 0" />
+    <parent link="chassis"/>
+    <child link="hokuyo" />
+    <axis xyz="0 1 0"/>
+  </joint>
+  <joint type="continuous" name="left_wheel_hinge">
+    <origin xyz="0 0.30 0" rpy="0 0 0" />
+    <parent link="chassis"/>
+    <child link="left_wheel" />
+    <axis xyz="0 1 0" rpy="0 0 0" />
+    <limit effort="10000" velocity="1000" />
+    <dynamics damping="1.0" friction="1.0" />
+  </joint>
+  <joint type="continuous" name="right_wheel_hinge">
+    <origin xyz="0 -0.30 0" rpy="0 0 0" />
+    <parent link="chassis"/>
+    <child link="right_wheel" />
+    <axis xyz="0 1 0" rpy="0 0 0" />
+    <limit effort="10000" velocity="1000" />
+    <dynamics damping="1.0" friction="1.0" />
+  </joint>
+<link name="camera">
+    <inertial>
+      <mass value="0.1"/>
+      <origin xyz="0 0 0" rpy="0 0 0"/>
+      <inertia
+        ixx="1e-6" ixy="0.0" ixz="0.0"
+        iyy="1e-6" iyz="0.0"
+        izz="1e-6"
+      />
+    </inertial>
+    <collision>
+      <origin xyz="0 0 0.1" rpy="0 0 0"/>
+      <geometry>
+        <box size="0.05 0.05 0.05"/>
+      </geometry>
+    </collision>
+    <visual>
+      <origin xyz="0 0 0.1" rpy="0 0 0"/>
+      <geometry>
+        <box size="0.05 0.05 0.05"/>
+      </geometry>
+    </visual>
+  </link>
+  <link name="hokuyo">
+    <inertial>
+      <mass value="1e-5"/>
+      <origin xyz="0 0 0" rpy="0 0 0"/>
+      <inertia
+        ixx="1e-6" ixy="0.0" ixz="0.0"
+        iyy="1e-6" iyz="0.0"
+        izz="1e-6"
+      />
+    </inertial>
+    <collision>
+      <origin xyz="0 0 0.12" rpy="0 0 0"/>
+      <geometry>
+        <box size="0.1 0.1 0.1"/>
+      </geometry>
+    </collision>
+    <visual>
+      <origin xyz="0 0 0.12" rpy="0 0 0"/>
+      <geometry>
+        <mesh filename="package://my_robot_urdf/meshes/hokuyo.dae"/>
+      </geometry>
+    </visual>
+  </link>
+  <link name="left_wheel">
+    <inertial>
+      <mass value="5"/>
+      <origin xyz="0 0 0" rpy="0 1.5707 1.5707"/>
+      <inertia
+        ixx="0.1" ixy="0.0" ixz="0.0"
+        iyy="0.1" iyz="0.0"
+        izz="0.1"
+      />
+    </inertial>
+    <collision>
+      <origin xyz="0 0 0" rpy="0 1.5707 1.5707"/>
+      <geometry>
+        <cylinder radius="0.1" length="0.05"/>
+      </geometry>
+    </collision>
+    <visual>
+      <origin xyz="0 0 0" rpy="0 1.5707 1.5707"/>
+      <geometry>
+        <cylinder radius="0.1" length="0.05"/>
+      </geometry>
+    </visual>
+  </link>
+  <link name="right_wheel">
+    <inertial>
+      <mass value="5"/>
+      <origin xyz="0 0 0" rpy="0 1.5707 1.5707"/>
+      <inertia
+        ixx="0.1" ixy="0.0" ixz="0.0"
+        iyy="0.1" iyz="0.0"
+        izz="0.1"
+      />
+    </inertial>
+    <collision>
+      <origin xyz="0 0 0" rpy="0 1.5707 1.5707"/>
+      <geometry>
+        <cylinder radius="0.1" length="0.05"/>
+      </geometry>
+    </collision>
+    <visual>
+      <origin xyz="0 0 0" rpy="0 1.5707 1.5707"/>
+      <geometry>
+        <cylinder radius="0.1" length="0.05"/>
+      </geometry>
+    </visual>
+  </link>
   <link name='chassis'>
     <pose>0 0 0.1 0 0 0</pose>
@@ -13,13 +161,37 @@
     </inertial>
     <collision name='collision'>
-      <origin xyz="0 0 0.05" rpy=" 0 0 0"/>
-      <geometry>
-        <cylinder length="0.2" radius="0.25"/>
+      <origin xyz="0 0 0.12" rpy=" 0 0 0"/>
+      <geometry>
+        <cylinder length="0.35" radius="0.25"/>
       </geometry>
     </collision>
     <visual name='chassis_visual'>
-      <origin xyz="0 0 0.05" rpy=" 0 0 0"/>
-      <geometry>
-       <cylinder length="0.2" radius="0.25"/>
+      <origin xyz="0 0 0.12" rpy=" 0 0 0"/>
+      <geometry>
+       <cylinder length="0.35" radius="0.25"/>
+      </geometry>
+    </visual>
+    <collision name='leftarm'>
+      <origin xyz="0.3 0.25 0.2" rpy="0 0 0"/>
+      <geometry>
+        <box size="0.6 0.04 0.09"/>
+      </geometry>
+    </collision>
+    <visual name='leftarm_visual'>
+      <origin xyz="0.3 0.25 0.2" rpy="0 0 0"/>
+      <geometry>
+        <box size="0.6 0.04 0.09"/>
+      </geometry>
+    </visual>
+    <collision name='rightarm'>
+      <origin xyz="0.3 -0.25 0.2" rpy="0 0 0"/>
+      <geometry>
+        <box size="0.6 0.04 0.09"/>
+      </geometry>
+    </collision>
+    <visual name='rightarm_visual'>
+      <origin xyz="0.3 -0.25 0.2" rpy="0 0 0"/>
+      <geometry>
+        <box size="0.6 0.04 0.09"/>
       </geometry>
     </visual>

Commit message: modified robot model

File: my_robot_urdf/urdf/robo.xacro (robot description, xacro)
@@ -14,4 +14,7 @@
     <material>Gazebo/Red</material>
   </gazebo>
+  <gazebo reference="head">
+    <material>Gazebo/Yellow</material>
+  </gazebo>
   <gazebo reference="leftarm">
     <material>Gazebo/Grey</material>
@@ -68,13 +71,13 @@
     </inertial>
     <collision>
-      <origin xyz="0 0 0.1" rpy="0 0 0"/>
-      <geometry>
-        <box size="0.05 0.05 0.05"/>
-      </geometry>
-    </collision>
-    <visual>
-      <origin xyz="0 0 0.1" rpy="0 0 0"/>
-      <geometry>
-        <box size="0.05 0.05 0.05"/>
+      <origin xyz="0.03 0 0.15" rpy="0 0 0"/>
+      <geometry>
+        <box size="0.06 0.05 0.05"/>
+      </geometry>
+    </collision>
+    <visual>
+      <origin xyz="0.03 0 0.15" rpy="0 0 0"/>
+      <geometry>
+        <box size="0.06 0.05 0.05"/>
       </geometry>
     </visual>
@@ -163,5 +166,5 @@
       <origin xyz="0 0 0.12" rpy=" 0 0 0"/>
       <geometry>
-        <cylinder length="0.35" radius="0.25"/>
+        <cylinder length="0.35" radius="0.28"/>
       </geometry>
     </collision>
@@ -169,29 +172,41 @@
       <origin xyz="0 0 0.12" rpy=" 0 0 0"/>
       <geometry>
-       <cylinder length="0.35" radius="0.25"/>
-      </geometry>
-    </visual>
-    <collision name='leftarm'>
-      <origin xyz="0.3 0.25 0.2" rpy="0 0 0"/>
-      <geometry>
-        <box size="0.6 0.04 0.09"/>
+       <cylinder length="0.35" radius="0.28"/>
+      </geometry>
+    </visual>
+    <collision name="head">
+      <origin xyz="0 0 0.3" rpy="0 0 0"/>
+      <geometry>
+        <sphere radius="0.15"/>
+      </geometry>
+    </collision>
+    <visual name="head_visual">
+      <origin xyz="0 0 0.3" rpy="0 0 0"/>
+      <geometry>
+        <sphere radius="0.15"/>
+      </geometry>
+    </visual>
+    <collision name="leftarm">
+      <origin xyz="0.4 0.25 0.06" rpy="0 0 0"/>
+      <geometry>
+        <box size="0.7 0.04 0.23"/>
       </geometry>
     </collision>
     <visual name='leftarm_visual'>
-      <origin xyz="0.3 0.25 0.2" rpy="0 0 0"/>
-      <geometry>
-        <box size="0.6 0.04 0.09"/>
-      </geometry>
-    </visual>
-    <collision name='rightarm'>
-      <origin xyz="0.3 -0.25 0.2" rpy="0 0 0"/>
-      <geometry>
-        <box size="0.6 0.04 0.09"/>
-      </geometry>
-    </collision>
-    <visual name='rightarm_visual'>
-      <origin xyz="0.3 -0.25 0.2" rpy="0 0 0"/>
-      <geometry>
-        <box size="0.6 0.04 0.09"/>
+      <origin xyz="0.4 0.25 0.06" rpy="0 0 0"/>
+      <geometry>
+        <box size="0.7 0.04 0.23"/>
+      </geometry>
+    </visual>
+    <collision name="rightarm">
+      <origin xyz="0.4 -0.25 0.06" rpy="0 0 0"/>
+      <geometry>
+        <box size="0.7 0.04 0.23"/>
+      </geometry>
+    </collision>
+    <visual name="rightarm_visual">
+      <origin xyz="0.4 -0.25 0.06" rpy="0 0 0"/>
+      <geometry>
+        <box size="0.7 0.04 0.23"/>
       </geometry>
     </visual>

Commit message: modified to spawn robot to assessment world

File: my_robot_urdf/urdf/robo.xacro (robot description, xacro)
@@ -71,5 +71,5 @@
     </inertial>
     <collision>
-      <origin xyz="0.03 0 0.15" rpy="0 0 0"/>
+      <origin xyz="0.01 0 0.15" rpy="0 0 0"/>
       <geometry>
         <box size="0.06 0.05 0.05"/>
@@ -77,5 +77,5 @@
     </collision>
     <visual>
-      <origin xyz="0.03 0 0.15" rpy="0 0 0"/>
+      <origin xyz="0.01 0 0.15" rpy="0 0 0"/>
       <geometry>
         <box size="0.06 0.05 0.05"/>
@@ -166,5 +166,5 @@
       <origin xyz="0 0 0.12" rpy=" 0 0 0"/>
       <geometry>
-        <cylinder length="0.35" radius="0.28"/>
+        <cylinder length="0.35" radius="0.25"/>
       </geometry>
     </collision>
@@ -172,5 +172,5 @@
       <origin xyz="0 0 0.12" rpy=" 0 0 0"/>
       <geometry>
-       <cylinder length="0.35" radius="0.28"/>
+       <cylinder length="0.35" radius="0.25"/>
       </geometry>
     </visual>
@@ -188,25 +188,25 @@
     </visual>
     <collision name="leftarm">
-      <origin xyz="0.4 0.25 0.06" rpy="0 0 0"/>
-      <geometry>
-        <box size="0.7 0.04 0.23"/>
+      <origin xyz="0.3 0.23 0.06" rpy="0 0 0"/>
+      <geometry>
+        <box size="0.5 0.03 0.23"/>
       </geometry>
     </collision>
     <visual name='leftarm_visual'>
-      <origin xyz="0.4 0.25 0.06" rpy="0 0 0"/>
-      <geometry>
-        <box size="0.7 0.04 0.23"/>
+      <origin xyz="0.3 0.23 0.06" rpy="0 0 0"/>
+      <geometry>
+        <box size="0.5 0.03 0.23"/>
       </geometry>
     </visual>
     <collision name="rightarm">
-      <origin xyz="0.4 -0.25 0.06" rpy="0 0 0"/>
-      <geometry>
-        <box size="0.7 0.04 0.23"/>
+      <origin xyz="0.3 -0.23 0.06" rpy="0 0 0"/>
+      <geometry>
+        <box size="0.5 0.03 0.23"/>
       </geometry>
     </collision>
     <visual name="rightarm_visual">
-      <origin xyz="0.4 -0.25 0.06" rpy="0 0 0"/>
-      <geometry>
-        <box size="0.7 0.04 0.23"/>
+      <origin xyz="0.3 -0.23 0.06" rpy="0 0 0"/>
+      <geometry>
+        <box size="0.5 0.03 0.23"/>
       </geometry>
     </visual>
